Commit message: bug修复

File: src/fw-mid/urdf/car1_fw-mid.xacro (robot description, xacro)
@@ -2,5 +2,5 @@
 <robot name="car1" xmlns:xacro="http://www.ros.org/wiki/xacro">
     <xacro:include filename="$(find fw-mid)/urdf/car1_macros.xacro" />
-    <link name="base_footprint">
+    <link name="car1_base_footprint">
         <!-- <visual>
             <geometry>
@@ -35,8 +35,8 @@
         </inertial>
     </link>
-    <joint name="base_link2base_footprint" type="fixed">
-        <parent link="base_footprint" />
+    <joint name="base_link2car1_base_footprint" type="fixed">
+        <parent link="car1_base_footprint" />
         <child link="base_link"/>
-        <origin xyz="0 0 0.032" />
+        <origin xyz="0 0 0.12" />
     </joint>
     <link name="left_steering_hinge">

File: src/fw-mid/urdf/car2_fw-mid.xacro (robot description, xacro)
@@ -2,5 +2,5 @@
 <robot name="car2" xmlns:xacro="http://www.ros.org/wiki/xacro">
     <xacro:include filename="$(find fw-mid)/urdf/car2_macros.xacro" />
-    <link name="base_footprint">
+    <link name="car2_base_footprint">
         <!-- <visual>
             <geometry>
@@ -35,8 +35,8 @@
         </inertial>
     </link>
-    <joint name="base_link2base_footprint" type="fixed">
-        <parent link="base_footprint" />
+    <joint name="base_link2car2_base_footprint" type="fixed">
+        <parent link="car2_base_footprint" />
         <child link="base_link"/>
-        <origin xyz="0 0 0.032" />
+        <origin xyz="0 0 0.12" />
     </joint>
     <link name="left_steering_hinge">

Commit message: bug修复

File: src/fw-mid/urdf/car1_fw-mid.xacro (robot description, xacro)
@@ -345,5 +345,5 @@
         <inertial>
         <mass value="0.001"/>
-        <origin xyz="0 0 0" rpy="0 0 0"/>
+        <origin xyz="0 0 0" rpy="0 0 3.14"/>
         <inertia ixx="0.0001" ixy="0.0" ixz="0.0" iyy="0.0001" iyz="0.0" izz="0.0001"/>
         </inertial>
@@ -357,5 +357,5 @@
         <gravity>true</gravity>
         <sensor type="ray" name="laser_livox">
-            <pose>0 0 0.04412 0 0 0</pose>
+            <pose>0 0 0.04412 0 0 3.1415926</pose>
             <visualize>true</visualize>
             <always_on>True</always_on>

File: src/fw-mid/urdf/car2_fw-mid.xacro (robot description, xacro)
@@ -357,5 +357,5 @@
         <gravity>true</gravity>
         <sensor type="ray" name="laser_livox">
-            <pose>0 0 0.04412 0 0 0</pose>
+            <pose>0 0 0.04412 0 0 3.1415926</pose>
             <visualize>true</visualize>
             <always_on>True</always_on>
